Commit message: added livox plugin

File: robots/descriptions/go2_description/xacro/robot.xacro (robot description, xacro)
@@ -10,4 +10,5 @@
     <xacro:include filename="$(find realsense2_description)/urdf/_d435.urdf.xacro"/>
     <xacro:include filename="$(find go2_description)/xacro/camera_gazebo.xacro"/>
+    <xacro:include filename="$(find ros2_livox_simulation)/urdf/mid360.xacro" />
     <!-- <xacro:stairs stairs="15" xpos="0" ypos="0" zpos="0" /> -->
     <!-- Rotor related joint and link is only for demonstrate location. -->
@@ -118,3 +119,6 @@
     </xacro:sensor_d435>
     <xacro:d435_gazebo_plugin camera_name="camera"/>
+    <xacro:mid360 name="livox" parent="trunk" topic="mid360">
+      <origin xyz="0 0 0.08" rpy="0 0 0"/>
+    </xacro:mid360>
 </robot>
